File: sango.sch (KiCad schematic (older format))
At the start: 23 parts

Commit message: add footprints for 0805 resistors
Parts:
- R? (x13): footprint (none) -> Resistor_SMD:R_0805_2012Metric_Pad1.15x1.40mm_HandSolder
Changed lines of the file:
@@
 F 0 "R?" V 4830 3450 50  0000 C CNN
 F 1 "10k" V 4750 3450 50  0000 C CNN
-F 2 "" V 4680 3450 50  0001 C CNN
+F 2 "Resistor_SMD:R_0805_2012Metric_Pad1.15x1.40mm_HandSolder" V 4680 3450 50  0001 C CNN
 F 3 "https://industrial.panasonic.com/cdbs/www-data/pdf/RDA0000/AOA0000C304.pdf" H 4750 3450 50  0001 C CNN
 F 4 "RES SMD 10K OHM 1% 1/8W 0805" H 4750 3450 50  0001 C CNN "Description"
@@
 F 0 "R?" V 4830 3600 50  0000 C CNN
 F 1 "10k" V 4750 3600 50  0000 C CNN
-F 2 "" V 4680 3600 50  0001 C CNN
+F 2 "Resistor_SMD:R_0805_2012Metric_Pad1.15x1.40mm_HandSolder" V 4680 3600 50  0001 C CNN
 F 3 "https://industrial.panasonic.com/cdbs/www-data/pdf/RDA0000/AOA0000C304.pdf" H 4750 3600 50  0001 C CNN
 F 4 "RES SMD 10K OHM 1% 1/8W 0805" H 4750 3600 50  0001 C CNN "Description"
@@
 F 0 "R?" V 4480 3950 50  0000 C CNN
 F 1 "5.1k" V 4400 3950 50  0000 C CNN
-F 2 "" V 4330 3950 50  0001 C CNN
+F 2 "Resistor_SMD:R_0805_2012Metric_Pad1.15x1.40mm_HandSolder" V 4330 3950 50  0001 C CNN
 F 3 "https://industrial.panasonic.com/cdbs/www-data/pdf/RDA0000/AOA0000C304.pdf" H 4400 3950 50  0001 C CNN
 F 4 "RES SMD 5.1K OHM 1% 1/8W 0805" H 4400 3950 50  0001 C CNN "Description"
@@
 F 0 "R?" V 4330 3950 50  0000 C CNN
 F 1 "5.1k" V 4250 3950 50  0000 C CNN
-F 2 "" V 4180 3950 50  0001 C CNN
+F 2 "Resistor_SMD:R_0805_2012Metric_Pad1.15x1.40mm_HandSolder" V 4180 3950 50  0001 C CNN
 F 3 "https://industrial.panasonic.com/cdbs/www-data/pdf/RDA0000/AOA0000C304.pdf" H 4250 3950 50  0001 C CNN
 F 4 "RES SMD 5.1K OHM 1% 1/8W 0805" H 4250 3950 50  0001 C CNN "Description"
@@
 F 0 "R?" V 5080 2350 50  0000 C CNN
 F 1 "10k" V 5000 2350 50  0000 C CNN
-F 2 "" V 4930 2350 50  0001 C CNN
+F 2 "Resistor_SMD:R_0805_2012Metric_Pad1.15x1.40mm_HandSolder" V 4930 2350 50  0001 C CNN
 F 3 "https://industrial.panasonic.com/cdbs/www-data/pdf/RDA0000/AOA0000C304.pdf" H 5000 2350 50  0001 C CNN
 F 4 "RES SMD 10K OHM 1% 1/8W 0805" H 5000 2350 50  0001 C CNN "Description"
@@
 F 0 "R?" V 5230 2350 50  0000 C CNN
 F 1 "10k" V 5150 2350 50  0000 C CNN
-F 2 "" V 5080 2350 50  0001 C CNN
+F 2 "Resistor_SMD:R_0805_2012Metric_Pad1.15x1.40mm_HandSolder" V 5080 2350 50  0001 C CNN
 F 3 "https://industrial.panasonic.com/cdbs/www-data/pdf/RDA0000/AOA0000C304.pdf" H 5150 2350 50  0001 C CNN
 F 4 "RES SMD 10K OHM 1% 1/8W 0805" H 5150 2350 50  0001 C CNN "Description"
@@
 F 0 "R?" V 4030 3250 50  0000 C CNN
 F 1 "5.1k" V 3950 3250 50  0000 C CNN
-F 2 "" V 3880 3250 50  0001 C CNN
+F 2 "Resistor_SMD:R_0805_2012Metric_Pad1.15x1.40mm_HandSolder" V 3880 3250 50  0001 C CNN
 F 3 "https://industrial.panasonic.com/cdbs/www-data/pdf/RDA0000/AOA0000C304.pdf" H 3950 3250 50  0001 C CNN
 F 4 "RES SMD 5.1K OHM 1% 1/8W 0805" H 3950 3250 50  0001 C CNN "Description"
@@
 F 0 "R?" V 4030 2850 50  0000 C CNN
 F 1 "35.7k" V 3950 2850 50  0000 C CNN
-F 2 "" V 3880 2850 50  0001 C CNN
+F 2 "Resistor_SMD:R_0805_2012Metric_Pad1.15x1.40mm_HandSolder" V 3880 2850 50  0001 C CNN
 F 3 "https://industrial.panasonic.com/cdbs/www-data/pdf/RDA0000/AOA0000C304.pdf" H 3950 2850 50  0001 C CNN
 F 4 "RES SMD 35.7K OHM 1% 1/8W 0805" H 3950 2850 50  0001 C CNN "Description"
@@
 F 0 "R?" V 2730 5150 50  0000 C CNN
 F 1 "1M" V 2650 5150 50  0000 C CNN
-F 2 "" V 2580 5150 50  0001 C CNN
+F 2 "Resistor_SMD:R_0805_2012Metric_Pad1.15x1.40mm_HandSolder" V 2580 5150 50  0001 C CNN
 F 3 "https://industrial.panasonic.com/cdbs/www-data/pdf/RDA0000/AOA0000C304.pdf" H 2650 5150 50  0001 C CNN
 F 4 "RES SMD 1M OHM 1% 1/8W 0805" H 2650 5150 50  0001 C CNN "Description"
@@
 F 0 "R?" V 8630 2350 50  0000 C CNN
 F 1 "10k" V 8550 2350 50  0000 C CNN
-F 2 "" V 8480 2350 50  0001 C CNN
+F 2 "Resistor_SMD:R_0805_2012Metric_Pad1.15x1.40mm_HandSolder" V 8480 2350 50  0001 C CNN
 F 3 "https://industrial.panasonic.com/cdbs/www-data/pdf/RDA0000/AOA0000C304.pdf" H 8550 2350 50  0001 C CNN
 F 4 "RES SMD 10K OHM 1% 1/8W 0805" H 8550 2350 50  0001 C CNN "Description"
@@
 F 0 "R?" V 8080 2350 50  0000 C CNN
 F 1 "150" V 8000 2350 50  0000 C CNN
-F 2 "" V 7930 2350 50  0001 C CNN
+F 2 "Resistor_SMD:R_0805_2012Metric_Pad1.15x1.40mm_HandSolder" V 7930 2350 50  0001 C CNN
 F 3 "https://industrial.panasonic.com/cdbs/www-data/pdf/RDA0000/AOA0000C304.pdf" H 8000 2350 50  0001 C CNN
 F 4 "RES SMD 150 OHM 1% 1/8W 0805" H 0   0   50  0001 C CNN "Description"
@@
 F 0 "R?" V 8230 2350 50  0000 C CNN
 F 1 "150" V 8150 2350 50  0000 C CNN
-F 2 "" V 8080 2350 50  0001 C CNN
+F 2 "Resistor_SMD:R_0805_2012Metric_Pad1.15x1.40mm_HandSolder" V 8080 2350 50  0001 C CNN
 F 3 "https://industrial.panasonic.com/cdbs/www-data/pdf/RDA0000/AOA0000C304.pdf" H 8150 2350 50  0001 C CNN
 F 4 "RES SMD 150 OHM 1% 1/8W 0805" H 0   0   50  0001 C CNN "Description"
@@
 F 0 "R?" V 9430 2350 50  0000 C CNN
 F 1 "90.9" V 9350 2350 50  0000 C CNN
-F 2 "" V 9280 2350 50  0001 C CNN
+F 2 "Resistor_SMD:R_0805_2012Metric_Pad1.15x1.40mm_HandSolder" V 9280 2350 50  0001 C CNN
 F 3 "https://industrial.panasonic.com/cdbs/www-data/pdf/RDA0000/AOA0000C304.pdf" H 9350 2350 50  0001 C CNN
 F 4 "RES SMD 90.9 OHM 1% 1/8W 0805" H 0   0   50  0001 C CNN "Description"

Commit message: add usb type-c receptable symbol modification to stdlibmods lib
Parts:
- removed J?: USB_C_Receptacle_USB2.0, symbol Connector:USB_C_Receptacle_USB2.0
- added J?: USB_C_Receptacle_USB2.0, symbol stdlibmods:USB_C_Receptacle_USB2.0
Changed lines of the file:
@@
 Wire Wire Line
 	4250 5400 4400 5400
-$Comp
-L Connector:USB_C_Receptacle_USB2.0 J?
-U 1 1 5BE5705F
-P 2850 3900
-F 0 "J?" H 2955 4767 50  0000 C CNN
-F 1 "USB_C_Receptacle_USB2.0" H 2955 4676 50  0000 C CNN
-F 2 "" H 3000 3900 50  0001 C CNN
-F 3 "https://www.usb.org/sites/default/files/documents/usb_type-c.zip" H 3000 3900 50  0001 C CNN
-	1    2850 3900
-	1    0    0    -1
-$EndComp
 Wire Wire Line
 	6200 2500 6200 2000
@@
 Wire Wire Line
 	9350 3000 9350 5400
+$Comp
+L stdlibmods:USB_C_Receptacle_USB2.0 J?
+U 1 1 5BF5DCD1
+P 2850 3900
+F 0 "J?" H 2955 4767 50  0000 C CNN
+F 1 "USB_C_Receptacle_USB2.0" H 2955 4676 50  0000 C CNN
+F 2 "" H 3000 3900 50  0001 C CNN
+F 3 "https://www.usb.org/sites/default/files/documents/usb_type-c.zip" H 3000 3900 50  0001 C CNN
+	1    2850 3900
+	1    0    0    -1
+$EndComp
 $EndSCHEMATC

Commit message: add jumpers for wired-or pfet gate operation
Parts:
- added J?: PFET_GATE, symbol stdlibmods:Conn_02x02_Odd_Even
Connections:
- net at Q?.1 (G), R?.1: now also J?.2 (Pin_2), J?.4 (Pin_4); no longer U?.10 (3.0_IND#), U?.9 (1.5_IND#)
- new net: J?.3 (Pin_3), U?.10 (3.0_IND#)
- new net: J?.1 (Pin_1), U?.9 (1.5_IND#)
Changed lines of the file:
@@
 $EndComp
-Wire Wire Line
-	7100 3450 8950 3450
-Wire Wire Line
-	7100 3600 8950 3600
-Wire Wire Line
-	8950 3600 8950 3450
-Wire Wire Line
-	8950 3450 8950 3000
-Connection ~ 8950 3450
 Wire Wire Line
 	6200 2000 8000 2000
@@
 	1    0    0    -1
 $EndComp
+$Comp
+L stdlibmods:Conn_02x02_Odd_Even J?
+U 1 1 5BF518D2
+P 8300 3450
+F 0 "J?" H 8350 3667 50  0000 C CNN
+F 1 "PFET_GATE" H 8350 3576 50  0000 C CNN
+F 2 "" H 8300 3450 50  0001 C CNN
+F 3 "~" H 8300 3450 50  0001 C CNN
+	1    8300 3450
+	1    0    0    -1
+$EndComp
+Wire Wire Line
+	8950 3000 8950 3450
+Wire Wire Line
+	8600 3600 8950 3600
+Wire Wire Line
+	8950 3450 8600 3450
+Connection ~ 8950 3450
+Wire Wire Line
+	8950 3450 8950 3600
+Wire Wire Line
+	8100 3450 7100 3450
+Wire Wire Line
+	7100 3600 8100 3600
 $EndSCHEMATC

Commit message: add decoupling 0.1uF for UTC2000, fill out fields for caps
Parts:
- added C?: 0.1u, Capacitor_SMD:C_0805_2012Metric_Pad1.15x1.40mm_HandSolder, symbol Device:C
- C?: footprint (none) -> Capacitor_SMD:C_0805_2012Metric_Pad1.15x1.40mm_HandSolder; Description (none) -> CAP CER 4.7PF 50V C0G/NP0 0805; Manufacturer (none) -> Samsung Electro-Mechanics; Manufacturer Part Number (none) -> CL21C4R7BBANNNC; Supplier (none) -> Digi-Key; Supplier Part Number (none) -> 1276-1832-1-ND
Connections:
- net +5V: now also C?.2
- net GND: now also C?.1
Other:
- moved on the sheet: J?
Changed lines of the file:
@@
 F 0 "C?" H 2335 5104 50  0000 R CNN
 F 1 "4.7n" H 2335 5195 50  0000 R CNN
-F 2 "" H 2488 5000 50  0001 C CNN
-F 3 "~" H 2450 5150 50  0001 C CNN
+F 2 "Capacitor_SMD:C_0805_2012Metric_Pad1.15x1.40mm_HandSolder" H 2488 5000 50  0001 C CNN
+F 3 "http://www.samsungsem.com/kr/support/product-search/mlcc/__icsFiles/afieldfile/2018/06/12/CL21C4R7BBANNNC.pdf" H 2450 5150 50  0001 C CNN
+F 4 "CAP CER 4.7PF 50V C0G/NP0 0805" H 0   0   50  0001 C CNN "Description"
+F 5 "Samsung Electro-Mechanics" H 0   0   50  0001 C CNN "Manufacturer"
+F 6 "CL21C4R7BBANNNC" H 0   0   50  0001 C CNN "Manufacturer Part Number"
+F 7 "Digi-Key" H 0   0   50  0001 C CNN "Supplier"
+F 8 "1276-1832-1-ND" H 0   0   50  0001 C CNN "Supplier Part Number"
 	1    2450 5150
 	1    0    0    1
@@
 	8150 2000 8150 2200
 Wire Wire Line
-	8150 2000 8550 2000
+	8150 2000 8350 2000
 Connection ~ 8150 2000
 $Comp
@@
 	9350 2000 9350 2200
 Wire Wire Line
-	9350 5400 6300 5400
+	9350 5400 8350 5400
 Connection ~ 6300 5400
 Wire Wire Line
@@
 L stdlibmods:Conn_02x02_Odd_Even J?
 U 1 1 5BF518D2
-P 8300 3450
-F 0 "J?" H 8350 3667 50  0000 C CNN
-F 1 "PFET_GATE" H 8350 3576 50  0000 C CNN
-F 2 "" H 8300 3450 50  0001 C CNN
-F 3 "~" H 8300 3450 50  0001 C CNN
-	1    8300 3450
+P 7600 3450
+F 0 "J?" H 7650 3100 50  0000 C CNN
+F 1 "PFET_GATE" H 7650 3200 50  0000 C CNN
+F 2 "" H 7600 3450 50  0001 C CNN
+F 3 "~" H 7600 3450 50  0001 C CNN
+	1    7600 3450
 	1    0    0    -1
 $EndComp
@@
 	8950 3000 8950 3450
 Wire Wire Line
-	8600 3600 8950 3600
-Wire Wire Line
-	8950 3450 8600 3450
+	7900 3600 8950 3600
+Wire Wire Line
+	8950 3450 7900 3450
 Connection ~ 8950 3450
 Wire Wire Line
 	8950 3450 8950 3600
 Wire Wire Line
-	8100 3450 7100 3450
-Wire Wire Line
-	7100 3600 8100 3600
+	7400 3450 7100 3450
+Wire Wire Line
+	7100 3600 7400 3600
+$Comp
+L Device:C C?
+U 1 1 5BF4E510
+P 8350 4200
+F 0 "C?" H 8235 4154 50  0000 R CNN
+F 1 "0.1u" H 8235 4245 50  0000 R CNN
+F 2 "Capacitor_SMD:C_0805_2012Metric_Pad1.15x1.40mm_HandSolder" H 8388 4050 50  0001 C CNN
+F 3 "http://www.samsungsem.com/kr/support/product-search/mlcc/__icsFiles/afieldfile/2018/07/23/CL21B104MBCNNNC.pdf" H 8350 4200 50  0001 C CNN
+F 4 "CAP CER 0.1UF 50V X7R 0805" H 0   0   50  0001 C CNN "Description"
+F 5 "Samsung Electro-Mechanics" H 0   0   50  0001 C CNN "Manufacturer"
+F 6 "CL21B104MBCNNNC" H 0   0   50  0001 C CNN "Manufacturer Part Number"
+F 7 "Digi-Key" H 0   0   50  0001 C CNN "Supplier"
+F 8 "1276-2450-1-ND" H 0   0   50  0001 C CNN "Supplier Part Number"
+	1    8350 4200
+	1    0    0    1
+$EndComp
+Wire Wire Line
+	8350 4050 8350 2000
+Connection ~ 8350 2000
+Wire Wire Line
+	8350 2000 8550 2000
+Wire Wire Line
+	8350 4350 8350 5400
+Connection ~ 8350 5400
+Wire Wire Line
+	8350 5400 6300 5400
 $EndSCHEMATC

Commit message: assign footprint for UTC2000
Parts:
- U?: footprint (none) -> microchip:UTC2000
Changed lines of the file:
@@
 F 0 "U?" H 6200 3250 50  0000 C CNN
 F 1 "UTC2000-I_MG" H 6200 3150 50  0000 C CNN
-F 2 "" H 4200 3700 50  0001 C CIN
+F 2 "microchip:UTC2000" H 4200 3700 50  0001 C CIN
 F 3 "http://ww1.microchip.com/downloads/en/DeviceDoc/UTC2000%20DS%2000001957C.pdf" H 6200 2400 50  0001 C CNN
 F 4 "Basic USB Type-C Controller" H 6200 2400 60  0001 C CNN "Description"

Commit message: assign 2mm diameter pad footprint to testpads
Parts:
- TP? (x3): footprint (none) -> TestPoint:TestPoint_Pad_D2.0mm
Changed lines of the file:
@@
 F 0 "TP?" H 5042 4127 50  0000 R CNN
 F 1 "OSC#" H 5042 4218 50  0000 R CNN
-F 2 "" H 5300 4100 50  0001 C CNN
+F 2 "TestPoint:TestPoint_Pad_D2.0mm" H 5300 4100 50  0001 C CNN
 F 3 "~" H 5300 4100 50  0001 C CNN
 	1    5100 4100
@@
 F 0 "TP?" H 7242 4127 50  0000 R CNN
 F 1 "LEGACY" H 7242 4218 50  0000 R CNN
-F 2 "" H 7500 4100 50  0001 C CNN
+F 2 "TestPoint:TestPoint_Pad_D2.0mm" H 7500 4100 50  0001 C CNN
 F 3 "~" H 7500 4100 50  0001 C CNN
 	1    7300 4100
@@
 F 0 "TP?" H 7242 2620 50  0000 R CNN
 F 1 "FAULT" H 7242 2529 50  0000 R CNN
-F 2 "" H 7500 2500 50  0001 C CNN
+F 2 "TestPoint:TestPoint_Pad_D2.0mm" H 7500 2500 50  0001 C CNN
 F 3 "~" H 7500 2500 50  0001 C CNN
 	1    7300 2500

Commit message: assign usbc receptable footprint & set fields
Parts:
- J?: footprint (none) -> amphenol:USB_C_Receptacle_Amphenol_12401598E4-2A; Description (none) -> CONN RCPT USB3.1 TYPEC SMD R/A; Manufacturer (none) -> Amphenol Commercial Products; Manufacturer Part Number (none) -> 12401598E4#2A; Supplier (none) -> Digi-Key; Supplier Part Number (none) -> 12401598E4#2ACT-ND
Changed lines of the file:
@@
 F 0 "J?" H 2955 4767 50  0000 C CNN
 F 1 "USB_C_Receptacle_USB2.0" H 2955 4676 50  0000 C CNN
-F 2 "" H 3000 3900 50  0001 C CNN
-F 3 "https://www.usb.org/sites/default/files/documents/usb_type-c.zip" H 3000 3900 50  0001 C CNN
+F 2 "amphenol:USB_C_Receptacle_Amphenol_12401598E4-2A" H 3000 3900 50  0001 C CNN
+F 3 "https://www.amphenol-icc.com/media/wysiwyg/files/drawing/12401598xxx2a.pdf" H 3000 3900 50  0001 C CNN
+F 4 "CONN RCPT USB3.1 TYPEC SMD R/A" H 0   0   50  0001 C CNN "Description"
+F 5 "Amphenol Commercial Products" H 0   0   50  0001 C CNN "Manufacturer"
+F 6 "12401598E4#2A" H 0   0   50  0001 C CNN "Manufacturer Part Number"
+F 7 "Digi-Key" H 0   0   50  0001 C CNN "Supplier"
+F 8 "12401598E4#2ACT-ND" H 0   0   50  0001 C CNN "Supplier Part Number"
 	1    2850 3900
 	1    0    0    -1

Commit message: assign jumper pin header footprint & set fields
Parts:
- J?: footprint (none) -> Connector_PinHeader_2.54mm:PinHeader_2x02_P2.54mm_Vertical; Description (none) -> CONN HEADER .100\" DUAL STR 4POS; Manufacturer (none) -> Sullins Connector Solutions; Manufacturer Part Number (none) -> PRPC002DAAN-RC; Supplier (none) -> Digi-Key; Supplier Part Number (none) -> S2011EC-02-ND
Changed lines of the file:
@@
 F 0 "J?" H 7650 3100 50  0000 C CNN
 F 1 "PFET_GATE" H 7650 3200 50  0000 C CNN
-F 2 "" H 7600 3450 50  0001 C CNN
-F 3 "~" H 7600 3450 50  0001 C CNN
+F 2 "Connector_PinHeader_2.54mm:PinHeader_2x02_P2.54mm_Vertical" H 7600 3450 50  0001 C CNN
+F 3 "https://drawings-pdf.s3.amazonaws.com/11636.pdf" H 7600 3450 50  0001 C CNN
+F 4 "CONN HEADER .100\" DUAL STR 4POS" H 0   0   50  0001 C CNN "Description"
+F 5 "Sullins Connector Solutions" H 0   0   50  0001 C CNN "Manufacturer"
+F 6 "PRPC002DAAN-RC" H 0   0   50  0001 C CNN "Manufacturer Part Number"
+F 7 "Digi-Key" H 0   0   50  0001 C CNN "Supplier"
+F 8 "S2011EC-02-ND" H 0   0   50  0001 C CNN "Supplier Part Number"
 	1    7600 3450
 	1    0    0    -1
