File: sango.sch (KiCad schematic (older format))
At the start: 25 parts

Commit message: assign LED footprints & set fields
Parts:
- D?: footprint (none) -> LED_SMD:LED_0805_2012Metric_Pad1.15x1.40mm_HandSolder; Description (none) -> LED YELLOW CLEAR 0805 SMD; Manufacturer (none) -> Wurth Electronics Inc.; Manufacturer Part Number (none) -> 150080YS75000; Supplier (none) -> Digi-Key; Supplier Part Number (none) -> 732-4987-1-ND
- D?: footprint (none) -> LED_SMD:LED_0805_2012Metric_Pad1.15x1.40mm_HandSolder; Description (none) -> LED RED CLEAR 0805 SMD; Manufacturer (none) -> Wurth Electronics Inc.; Manufacturer Part Number (none) -> 150080RS75000; Supplier (none) -> Digi-Key; Supplier Part Number (none) -> 732-4984-1-ND
- D?: footprint (none) -> LED_SMD:LED_0805_2012Metric_Pad1.15x1.40mm_HandSolder; Description (none) -> LED BLUE CLEAR 0805 SMD; Manufacturer (none) -> Wurth Electronics Inc.; Manufacturer Part Number (none) -> 150080BS75000; Supplier (none) -> Digi-Key; Supplier Part Number (none) -> 732-4982-1-ND
Changed lines of the file:
@@
 F 0 "D?" H 7650 2800 50  0000 C CNN
 F 1 "YELLOW" H 7650 2900 50  0000 C CNN
-F 2 "" H 7650 3000 50  0001 C CNN
-F 3 "~" H 7650 3000 50  0001 C CNN
+F 2 "LED_SMD:LED_0805_2012Metric_Pad1.15x1.40mm_HandSolder" H 7650 3000 50  0001 C CNN
+F 3 "https://katalog.we-online.de/led/datasheet/150080YS75000.pdf" H 7650 3000 50  0001 C CNN
+F 4 "LED YELLOW CLEAR 0805 SMD" H 0   0   50  0001 C CNN "Description"
+F 5 "Wurth Electronics Inc." H 0   0   50  0001 C CNN "Manufacturer"
+F 6 "150080YS75000" H 0   0   50  0001 C CNN "Manufacturer Part Number"
+F 7 "Digi-Key" H 0   0   50  0001 C CNN "Supplier"
+F 8 "732-4987-1-ND" H 0   0   50  0001 C CNN "Supplier Part Number"
 	1    7650 3000
 	1    0    0    -1
@@
 F 0 "D?" H 7650 2650 50  0000 C CNN
 F 1 "RED" H 7650 2750 50  0000 C CNN
-F 2 "" H 7650 2850 50  0001 C CNN
-F 3 "~" H 7650 2850 50  0001 C CNN
+F 2 "LED_SMD:LED_0805_2012Metric_Pad1.15x1.40mm_HandSolder" H 7650 2850 50  0001 C CNN
+F 3 "https://katalog.we-online.de/led/datasheet/150080RS75000.pdf" H 7650 2850 50  0001 C CNN
+F 4 "LED RED CLEAR 0805 SMD" H 0   0   50  0001 C CNN "Description"
+F 5 "Wurth Electronics Inc." H 0   0   50  0001 C CNN "Manufacturer"
+F 6 "150080RS75000" H 0   0   50  0001 C CNN "Manufacturer Part Number"
+F 7 "Digi-Key" H 0   0   50  0001 C CNN "Supplier"
+F 8 "732-4984-1-ND" H 0   0   50  0001 C CNN "Supplier Part Number"
 	1    7650 2850
 	1    0    0    1
@@
 F 0 "D?" H 9350 2650 50  0000 C CNN
 F 1 "BLUE" H 9350 2750 50  0000 C CNN
-F 2 "" H 9350 2850 50  0001 C CNN
-F 3 "~" H 9350 2850 50  0001 C CNN
+F 2 "LED_SMD:LED_0805_2012Metric_Pad1.15x1.40mm_HandSolder" H 9350 2850 50  0001 C CNN
+F 3 "https://katalog.we-online.de/led/datasheet/150080BS75000.pdf" H 9350 2850 50  0001 C CNN
+F 4 "LED BLUE CLEAR 0805 SMD" H 0   0   50  0001 C CNN "Description"
+F 5 "Wurth Electronics Inc." H 0   0   50  0001 C CNN "Manufacturer"
+F 6 "150080BS75000" H 0   0   50  0001 C CNN "Manufacturer Part Number"
+F 7 "Digi-Key" H 0   0   50  0001 C CNN "Supplier"
+F 8 "732-4982-1-ND" H 0   0   50  0001 C CNN "Supplier Part Number"
 	1    9350 2850
 	0    -1   -1   0

Commit message: annotate schematic
Parts:
- J1: renamed from J?; value USB_C_Receptacle_USB2.0 -> USB-C
- gave numbers to parts that had none: 24
Changed lines of the file:
@@
 $EndDescr
 $Comp
-L power:GND #PWR?
+L power:GND #PWR0101
 U 1 1 5A5454A8
 P 6200 5600
-F 0 "#PWR?" H 6200 5350 50  0001 C CNN
+F 0 "#PWR0101" H 6200 5350 50  0001 C CNN
 F 1 "GND" H 6200 5450 50  0000 C CNN
 F 2 "" H 6200 5600 50  0001 C CNN
@@
 	6100 3800 6100 5400
 $Comp
-L power:+5V #PWR?
+L power:+5V #PWR0102
 U 1 1 5A5454F9
 P 6200 1800
-F 0 "#PWR?" H 6200 1650 50  0001 C CNN
+F 0 "#PWR0102" H 6200 1650 50  0001 C CNN
 F 1 "+5V" H 6200 1940 50  0000 C CNN
 F 2 "" H 6200 1800 50  0001 C CNN
@@
 $EndComp
 $Comp
-L Device:R R?
+L Device:R R6
 U 1 1 5A545653
 P 4750 3450
-F 0 "R?" V 4830 3450 50  0000 C CNN
+F 0 "R6" V 4830 3450 50  0000 C CNN
 F 1 "10k" V 4750 3450 50  0000 C CNN
 F 2 "Resistor_SMD:R_0805_2012Metric_Pad1.15x1.40mm_HandSolder" V 4680 3450 50  0001 C CNN
@@
 $EndComp
 $Comp
-L Device:R R?
+L Device:R R7
 U 1 1 5A545694
 P 4750 3600
-F 0 "R?" V 4830 3600 50  0000 C CNN
+F 0 "R7" V 4830 3600 50  0000 C CNN
 F 1 "10k" V 4750 3600 50  0000 C CNN
 F 2 "Resistor_SMD:R_0805_2012Metric_Pad1.15x1.40mm_HandSolder" V 4680 3600 50  0001 C CNN
@@
 	4900 3600 5300 3600
 $Comp
-L Device:R R?
+L Device:R R5
 U 1 1 5A545718
 P 4400 3950
-F 0 "R?" V 4480 3950 50  0000 C CNN
+F 0 "R5" V 4480 3950 50  0000 C CNN
 F 1 "5.1k" V 4400 3950 50  0000 C CNN
 F 2 "Resistor_SMD:R_0805_2012Metric_Pad1.15x1.40mm_HandSolder" V 4330 3950 50  0001 C CNN
@@
 	4400 3600 4400 3800
 $Comp
-L Device:R R?
+L Device:R R4
 U 1 1 5A545776
 P 4250 3950
-F 0 "R?" V 4330 3950 50  0000 C CNN
+F 0 "R4" V 4330 3950 50  0000 C CNN
 F 1 "5.1k" V 4250 3950 50  0000 C CNN
 F 2 "Resistor_SMD:R_0805_2012Metric_Pad1.15x1.40mm_HandSolder" V 4180 3950 50  0001 C CNN
@@
 Connection ~ 6100 5400
 $Comp
-L Device:R R?
+L Device:R R8
 U 1 1 5A54597B
 P 5000 2350
-F 0 "R?" V 5080 2350 50  0000 C CNN
+F 0 "R8" V 5080 2350 50  0000 C CNN
 F 1 "10k" V 5000 2350 50  0000 C CNN
 F 2 "Resistor_SMD:R_0805_2012Metric_Pad1.15x1.40mm_HandSolder" V 4930 2350 50  0001 C CNN
@@
 $EndComp
 $Comp
-L Device:R R?
+L Device:R R9
 U 1 1 5A5459D2
 P 5150 2350
-F 0 "R?" V 5230 2350 50  0000 C CNN
+F 0 "R9" V 5230 2350 50  0000 C CNN
 F 1 "10k" V 5150 2350 50  0000 C CNN
 F 2 "Resistor_SMD:R_0805_2012Metric_Pad1.15x1.40mm_HandSolder" V 5080 2350 50  0001 C CNN
@@
 Connection ~ 5150 2000
 $Comp
-L Device:R R?
+L Device:R R3
 U 1 1 5A545D7A
 P 3950 3250
-F 0 "R?" V 4030 3250 50  0000 C CNN
+F 0 "R3" V 4030 3250 50  0000 C CNN
 F 1 "5.1k" V 3950 3250 50  0000 C CNN
 F 2 "Resistor_SMD:R_0805_2012Metric_Pad1.15x1.40mm_HandSolder" V 3880 3250 50  0001 C CNN
@@
 	3950 3050 5300 3050
 $Comp
-L Device:R R?
+L Device:R R2
 U 1 1 5A545E3E
 P 3950 2850
-F 0 "R?" V 4030 2850 50  0000 C CNN
+F 0 "R2" V 4030 2850 50  0000 C CNN
 F 1 "35.7k" V 3950 2850 50  0000 C CNN
 F 2 "Resistor_SMD:R_0805_2012Metric_Pad1.15x1.40mm_HandSolder" V 3880 2850 50  0001 C CNN
@@
 	6200 2500 6200 2000
 $Comp
-L Device:R R?
+L Device:R R1
 U 1 1 5BE75FE5
 P 2650 5150
-F 0 "R?" V 2730 5150 50  0000 C CNN
+F 0 "R1" V 2730 5150 50  0000 C CNN
 F 1 "1M" V 2650 5150 50  0000 C CNN
 F 2 "Resistor_SMD:R_0805_2012Metric_Pad1.15x1.40mm_HandSolder" V 2580 5150 50  0001 C CNN
@@
 $EndComp
 $Comp
-L Device:C C?
+L Device:C C1
 U 1 1 5BE76CD8
 P 2450 5150
-F 0 "C?" H 2335 5104 50  0000 R CNN
+F 0 "C1" H 2335 5104 50  0000 R CNN
 F 1 "4.7n" H 2335 5195 50  0000 R CNN
 F 2 "Capacitor_SMD:C_0805_2012Metric_Pad1.15x1.40mm_HandSolder" H 2488 5000 50  0001 C CNN
@@
 	2850 5400 3950 5400
 $Comp
-L microchip:UTC2000-I_MG U?
+L microchip:UTC2000-I_MG U1
 U 1 1 5BE535AB
 P 6200 3150
-F 0 "U?" H 6200 3250 50  0000 C CNN
+F 0 "U1" H 6200 3250 50  0000 C CNN
 F 1 "UTC2000-I_MG" H 6200 3150 50  0000 C CNN
 F 2 "microchip:UTC2000" H 4200 3700 50  0001 C CIN
@@
 $EndComp
 $Comp
-L Transistor_FET:NTR2101P Q?
+L Transistor_FET:NTR2101P Q1
 U 1 1 5BE8FFD4
 P 8950 2100
-F 0 "Q?" V 9293 2100 50  0000 C CNN
+F 0 "Q1" V 9293 2100 50  0000 C CNN
 F 1 "NTR2101P" V 9202 2100 50  0000 C CNN
 F 2 "Package_TO_SOT_SMD:SOT-23" H 9150 2025 50  0001 L CIN
@@
 Connection ~ 6200 2000
 $Comp
-L Device:R R?
+L Device:R R12
 U 1 1 5BE95889
 P 8550 2350
-F 0 "R?" V 8630 2350 50  0000 C CNN
+F 0 "R12" V 8630 2350 50  0000 C CNN
 F 1 "10k" V 8550 2350 50  0000 C CNN
 F 2 "Resistor_SMD:R_0805_2012Metric_Pad1.15x1.40mm_HandSolder" V 8480 2350 50  0001 C CNN
@@
 	8950 3000 8950 2300
 $Comp
-L Connector:TestPoint TP?
+L Connector:TestPoint TP1
 U 1 1 5BF445E0
 P 5100 4100
-F 0 "TP?" H 5042 4127 50  0000 R CNN
+F 0 "TP1" H 5042 4127 50  0000 R CNN
 F 1 "OSC#" H 5042 4218 50  0000 R CNN
 F 2 "TestPoint:TestPoint_Pad_D2.0mm" H 5300 4100 50  0001 C CNN
@@
 	5100 3250 5100 4100
 $Comp
-L Connector:TestPoint TP?
+L Connector:TestPoint TP3
 U 1 1 5BF45B7A
 P 7300 4100
-F 0 "TP?" H 7242 4127 50  0000 R CNN
+F 0 "TP3" H 7242 4127 50  0000 R CNN
 F 1 "LEGACY" H 7242 4218 50  0000 R CNN
 F 2 "TestPoint:TestPoint_Pad_D2.0mm" H 7500 4100 50  0001 C CNN
@@
 	6200 2000 6200 1800
 $Comp
-L Connector:TestPoint TP?
+L Connector:TestPoint TP2
 U 1 1 5BF5A8B0
 P 7300 2500
-F 0 "TP?" H 7242 2620 50  0000 R CNN
+F 0 "TP2" H 7242 2620 50  0000 R CNN
 F 1 "FAULT" H 7242 2529 50  0000 R CNN
 F 2 "TestPoint:TestPoint_Pad_D2.0mm" H 7500 2500 50  0001 C CNN
@@
 	7300 2700 7300 2500
 $Comp
-L Device:LED D?
+L Device:LED D2
 U 1 1 5BF5E104
 P 7650 3000
-F 0 "D?" H 7650 2800 50  0000 C CNN
+F 0 "D2" H 7650 2800 50  0000 C CNN
 F 1 "YELLOW" H 7650 2900 50  0000 C CNN
 F 2 "LED_SMD:LED_0805_2012Metric_Pad1.15x1.40mm_HandSolder" H 7650 3000 50  0001 C CNN
@@
 $EndComp
 $Comp
-L Device:LED D?
+L Device:LED D1
 U 1 1 5BF5E569
 P 7650 2850
-F 0 "D?" H 7650 2650 50  0000 C CNN
+F 0 "D1" H 7650 2650 50  0000 C CNN
 F 1 "RED" H 7650 2750 50  0000 C CNN
 F 2 "LED_SMD:LED_0805_2012Metric_Pad1.15x1.40mm_HandSolder" H 7650 2850 50  0001 C CNN
@@
 	7500 3000 7100 3000
 $Comp
-L Device:R R?
+L Device:R R10
 U 1 1 5BF67E3A
 P 8000 2350
-F 0 "R?" V 8080 2350 50  0000 C CNN
+F 0 "R10" V 8080 2350 50  0000 C CNN
 F 1 "150" V 8000 2350 50  0000 C CNN
 F 2 "Resistor_SMD:R_0805_2012Metric_Pad1.15x1.40mm_HandSolder" V 7930 2350 50  0001 C CNN
@@
 Connection ~ 8150 2000
 $Comp
-L Device:R R?
+L Device:R R11
 U 1 1 5BF78175
 P 8150 2350
-F 0 "R?" V 8230 2350 50  0000 C CNN
+F 0 "R11" V 8230 2350 50  0000 C CNN
 F 1 "150" V 8150 2350 50  0000 C CNN
 F 2 "Resistor_SMD:R_0805_2012Metric_Pad1.15x1.40mm_HandSolder" V 8080 2350 50  0001 C CNN
@@
 $EndComp
 $Comp
-L Device:LED D?
+L Device:LED D3
 U 1 1 5BF7A803
 P 9350 2850
-F 0 "D?" H 9350 2650 50  0000 C CNN
+F 0 "D3" H 9350 2650 50  0000 C CNN
 F 1 "BLUE" H 9350 2750 50  0000 C CNN
 F 2 "LED_SMD:LED_0805_2012Metric_Pad1.15x1.40mm_HandSolder" H 9350 2850 50  0001 C CNN
@@
 	6200 5400 6300 5400
 $Comp
-L Device:R R?
+L Device:R R13
 U 1 1 5BF89938
 P 9350 2350
-F 0 "R?" V 9430 2350 50  0000 C CNN
+F 0 "R13" V 9430 2350 50  0000 C CNN
 F 1 "90.9" V 9350 2350 50  0000 C CNN
 F 2 "Resistor_SMD:R_0805_2012Metric_Pad1.15x1.40mm_HandSolder" V 9280 2350 50  0001 C CNN
@@
 	9350 3000 9350 5400
 $Comp
-L stdlibmods:USB_C_Receptacle_USB2.0 J?
+L stdlibmods:USB_C_Receptacle_USB2.0 J1
 U 1 1 5BF5DCD1
 P 2850 3900
-F 0 "J?" H 2955 4767 50  0000 C CNN
-F 1 "USB_C_Receptacle_USB2.0" H 2955 4676 50  0000 C CNN
+F 0 "J1" H 2955 4767 50  0000 C CNN
+F 1 "USB-C" H 2955 4676 50  0000 C CNN
 F 2 "amphenol:USB_C_Receptacle_Amphenol_12401598E4-2A" H 3000 3900 50  0001 C CNN
 F 3 "https://www.amphenol-icc.com/media/wysiwyg/files/drawing/12401598xxx2a.pdf" H 3000 3900 50  0001 C CNN
@@
 $EndComp
 $Comp
-L stdlibmods:Conn_02x02_Odd_Even J?
+L stdlibmods:Conn_02x02_Odd_Even J2
 U 1 1 5BF518D2
 P 7600 3450
-F 0 "J?" H 7650 3100 50  0000 C CNN
+F 0 "J2" H 7650 3100 50  0000 C CNN
 F 1 "PFET_GATE" H 7650 3200 50  0000 C CNN
 F 2 "Connector_PinHeader_2.54mm:PinHeader_2x02_P2.54mm_Vertical" H 7600 3450 50  0001 C CNN
@@
 	7100 3600 7400 3600
 $Comp
-L Device:C C?
+L Device:C C2
 U 1 1 5BF4E510
 P 8350 4200
-F 0 "C?" H 8235 4154 50  0000 R CNN
+F 0 "C2" H 8235 4154 50  0000 R CNN
 F 1 "0.1u" H 8235 4245 50  0000 R CNN
 F 2 "Capacitor_SMD:C_0805_2012Metric_Pad1.15x1.40mm_HandSolder" H 8388 4050 50  0001 C CNN

Commit message: initial layout
- add kicad_pcb-bak to gitignore
- switch LED names for adding to silkscreen
Parts:
- D1: value RED -> CONN
- D2: value YELLOW -> UP/DN
- D3: value BLUE -> OUT
Changed lines of the file:
@@
 P 7650 3000
 F 0 "D2" H 7650 2800 50  0000 C CNN
-F 1 "YELLOW" H 7650 2900 50  0000 C CNN
+F 1 "UP/DN" H 7650 2900 50  0000 C CNN
 F 2 "LED_SMD:LED_0805_2012Metric_Pad1.15x1.40mm_HandSolder" H 7650 3000 50  0001 C CNN
 F 3 "https://katalog.we-online.de/led/datasheet/150080YS75000.pdf" H 7650 3000 50  0001 C CNN
@@
 P 7650 2850
 F 0 "D1" H 7650 2650 50  0000 C CNN
-F 1 "RED" H 7650 2750 50  0000 C CNN
+F 1 "CONN" H 7650 2750 50  0000 C CNN
 F 2 "LED_SMD:LED_0805_2012Metric_Pad1.15x1.40mm_HandSolder" H 7650 2850 50  0001 C CNN
 F 3 "https://katalog.we-online.de/led/datasheet/150080RS75000.pdf" H 7650 2850 50  0001 C CNN
@@
 P 9350 2850
 F 0 "D3" H 9350 2650 50  0000 C CNN
-F 1 "BLUE" H 9350 2750 50  0000 C CNN
+F 1 "OUT" H 9350 2750 50  0000 C CNN
 F 2 "LED_SMD:LED_0805_2012Metric_Pad1.15x1.40mm_HandSolder" H 9350 2850 50  0001 C CNN
 F 3 "https://katalog.we-online.de/led/datasheet/150080BS75000.pdf" H 9350 2850 50  0001 C CNN

Commit message: separate current schematic into 'USB-C Power' sheet
Parts:
- removed C1: 4.7n, Capacitor_SMD:C_0805_2012Metric_Pad1.15x1.40mm_HandSolder, symbol Device:C
- removed C2: 0.1u, Capacitor_SMD:C_0805_2012Metric_Pad1.15x1.40mm_HandSolder, symbol Device:C
- removed D1: CONN, LED_SMD:LED_0805_2012Metric_Pad1.15x1.40mm_HandSolder, symbol Device:LED
- removed D2: UP/DN, LED_SMD:LED_0805_2012Metric_Pad1.15x1.40mm_HandSolder, symbol Device:LED
- removed D3: OUT, LED_SMD:LED_0805_2012Metric_Pad1.15x1.40mm_HandSolder, symbol Device:LED
- removed J1: USB-C, amphenol:USB_C_Receptacle_Amphenol_12401598E4-2A, symbol stdlibmods:USB_C_Receptacle_USB2.0
- removed J2: PFET_GATE, Connector_PinHeader_2.54mm:PinHeader_2x02_P2.54mm_Vertical, symbol stdlibmods:Conn_02x02_Odd_Even
- removed Q1: NTR2101P, Package_TO_SOT_SMD:SOT-23, symbol Transistor_FET:NTR2101P
- removed R1: 1M, Resistor_SMD:R_0805_2012Metric_Pad1.15x1.40mm_HandSolder, symbol Device:R
- removed R10, R11: 150, Resistor_SMD:R_0805_2012Metric_Pad1.15x1.40mm_HandSolder, symbol Device:R
- removed R12, R6, R7, R8, R9: 10k, Resistor_SMD:R_0805_2012Metric_Pad1.15x1.40mm_HandSolder, symbol Device:R
- removed R13: 90.9, Resistor_SMD:R_0805_2012Metric_Pad1.15x1.40mm_HandSolder, symbol Device:R
- removed R2: 35.7k, Resistor_SMD:R_0805_2012Metric_Pad1.15x1.40mm_HandSolder, symbol Device:R
- removed R3, R4, R5: 5.1k, Resistor_SMD:R_0805_2012Metric_Pad1.15x1.40mm_HandSolder, symbol Device:R
- removed TP1: OSC#, TestPoint:TestPoint_Pad_D2.0mm, symbol Connector:TestPoint
- removed TP2: FAULT, TestPoint:TestPoint_Pad_D2.0mm, symbol Connector:TestPoint
- removed TP3: LEGACY, TestPoint:TestPoint_Pad_D2.0mm, symbol Connector:TestPoint
- removed U1: UTC2000-I_MG, microchip:UTC2000, symbol microchip:UTC2000-I_MG
Connections:
- net labels removed: +5V, GND
- wire segments 85 -> 0
- no-connect marks 6 -> 0
