File: sango.kicad_pcb (KiCad board)
At the start: 2 copper layers, 32 x 39 mm, 25 parts, among them J1 USB-C, J2 PFET_GATE, Q1 NTR2101P, U1 UTC2000-I_MG

Commit message: added rules for 4-layer OSHpark fab
Other:
- copper layers 2 -> 4
- net class Default: clearance 0.2 -> 0.1524; trace_width 0.25 -> 0.1524; via_dia 0.8 -> 0.6858; via_drill 0.4 -> 0.3302
- rule trace_clearance: 0.2 -> 0.1524
- rule trace_min: 0.2 -> 0.1524
- rule via_min_drill: 0.3 -> 0.3302
- rule via_min_size: 0.4 -> 0.6858
Changed lines of the file:
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@@
   (layers
     (0 F.Cu signal)
+    (1 In1.Cu signal)
+    (2 In2.Cu signal)
     (31 B.Cu signal)
-    (32 B.Adhes user)
-    (33 F.Adhes user)
     (34 B.Paste user)
     (35 F.Paste user)
@@
     (38 B.Mask user)
     (39 F.Mask user)
-    (40 Dwgs.User user)
-    (41 Cmts.User user)
-    (42 Eco1.User user)
-    (43 Eco2.User user)
     (44 Edge.Cuts user)
     (45 Margin user)
     (46 B.CrtYd user)
     (47 F.CrtYd user)
-    (48 B.Fab user)
-    (49 F.Fab user)
   )
   (setup
-    (last_trace_width 0.25)
-    (trace_clearance 0.2)
+    (last_trace_width 0.1524)
+    (trace_clearance 0.1524)
     (zone_clearance 0.508)
     (zone_45_only no)
-    (trace_min 0.2)
+    (trace_min 0.1524)
     (segment_width 0.2)
     (edge_width 0.15)
-    (via_size 0.8)
-    (via_drill 0.4)
-    (via_min_size 0.4)
-    (via_min_drill 0.3)
-    (uvia_size 0.3)
-    (uvia_drill 0.1)
+    (via_size 0.6858)
+    (via_drill 0.3302)
+    (via_min_size 0.6858)
+    (via_min_drill 0.3302)
+    (uvia_size 0.6858)
+    (uvia_drill 0.3302)
     (uvias_allowed no)
     (uvia_min_size 0.2)
@@
   (net 30 "Net-(U1-Pad15)")
   (net_class Default "This is the default net class."
-    (clearance 0.2)
-    (trace_width 0.25)
-    (via_dia 0.8)
-    (via_drill 0.4)
-    (uvia_dia 0.3)
-    (uvia_drill 0.1)
+    (clearance 0.1524)
+    (trace_width 0.1524)
+    (via_dia 0.6858)
+    (via_drill 0.3302)
+    (uvia_dia 0.6858)
+    (uvia_drill 0.3302)
+    (diff_pair_gap 0.1524)
+    (diff_pair_width 0.1524)
     (add_net +5V)
     (add_net GND)

Commit message: init 4-layer layout
- TODO: expand trace thickness past minimum
- TODO: review whether placing vias on pads is ok
- TODO: add silkscreen indicating which jumper is which
- TODO: board graphics
Parts:
- turned D1 to 180 degrees
Routing:
- net Net-(C1-Pad2): track 0.00 -> 34.2 mm
- net Net-(J2-Pad1): track 0.00 -> 21.4 mm
- net Net-(J2-Pad3): track 0.00 -> 17.8 mm
- net Net-(TP3-Pad1): track 0.00 -> 17.2 mm, vias 0 -> 2
- net Net-(J2-Pad2): track 0.00 -> 16.7 mm
- net Net-(J1-PadB5): track 0.00 -> 15.9 mm, vias 0 -> 2
- net Net-(D1-Pad1): track 0.00 -> 14.6 mm
- net Net-(TP2-Pad1): track 0.00 -> 14.5 mm, vias 0 -> 2
- net Net-(D2-Pad1): track 0.00 -> 14.5 mm
- net +5V: track 0.00 -> 12.8 mm, vias 0 -> 12
- net Net-(J1-PadA5): track 0.00 -> 10.9 mm
- net Net-(R2-Pad1): track 0.00 -> 9.66 mm
- net Net-(TP1-Pad1): track 0.00 -> 7.39 mm
- net GND: track 0.00 -> 6.84 mm, vias 0 -> 12
- net Net-(R9-Pad2): track 0.00 -> 6.04 mm
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- added copper zone on In2.Cu, net +5V
- added copper zone on In1.Cu, net GND
- added copper zone on In2.Cu, net Net-(Q1-Pad3)
