File: ldo-p12V.sch (KiCad schematic (older format))
At the start: 8 parts

Commit message: update resistor BOM for ldo sheets
Parts:
- R?: Description (none) -> RES SMD 121K OHM 1% 1/8W 0805; Manufacturer Part Number ERJ-6ENF1004V -> ERJ-6ENF1213V; Supplier Part Number P1.00MCCT-ND -> P121KCCT-ND
- R? (x2): Description (none) -> RES SMD 49.9K OHM 1% 1/8W 0805; Manufacturer Part Number ERJ-6ENF1004V -> ERJ-6ENF4992V; Supplier Part Number P1.00MCCT-ND -> P49.9KCCT-ND
- R?: Description (none) -> RES SMD 1.82M OHM 1% 1/8W 0805; Manufacturer Part Number ERJ-6ENF1004V -> ERJ-6ENF1824V; Supplier Part Number P1.00MCCT-ND -> P1.82BTCT-ND
- R?: Description (none) -> RES SMD 432K OHM 1% 1/8W 0805; Manufacturer Part Number ERJ-6ENF1004V -> ERJ-6ENF4323V; Supplier Part Number P1.00MCCT-ND -> P432KCCT-ND
Changed lines of the file:
@@
 F 2 "Resistor_SMD:R_0805_2012Metric_Pad1.15x1.40mm_HandSolder" V 4480 4400 50  0001 C CNN
 F 3 "https://industrial.panasonic.com/cdbs/www-data/pdf/RDA0000/AOA0000C304.pdf" H 4550 4400 50  0001 C CNN
-F 4 "" H 4550 4400 50  0001 C CNN "Description"
+F 4 "RES SMD 121K OHM 1% 1/8W 0805" H 4550 4400 50  0001 C CNN "Description"
 F 5 "Panasonic Electronic Components" H 4550 4400 50  0001 C CNN "Manufacturer"
-F 6 "ERJ-6ENF1004V" H 4550 4400 50  0001 C CNN "Manufacturer Part Number"
+F 6 "ERJ-6ENF1213V" H 4550 4400 50  0001 C CNN "Manufacturer Part Number"
 F 7 "Digi-Key" H 4550 4400 50  0001 C CNN "Supplier"
-F 8 "P1.00MCCT-ND" H 4550 4400 50  0001 C CNN "Supplier Part Number"
+F 8 "P121KCCT-ND" H 4550 4400 50  0001 C CNN "Supplier Part Number"
 	1    4550 4400
 	1    0    0    1
@@
 F 2 "Resistor_SMD:R_0805_2012Metric_Pad1.15x1.40mm_HandSolder" V 6380 4400 50  0001 C CNN
 F 3 "https://industrial.panasonic.com/cdbs/www-data/pdf/RDA0000/AOA0000C304.pdf" H 6450 4400 50  0001 C CNN
-F 4 "" H 6450 4400 50  0001 C CNN "Description"
+F 4 "RES SMD 49.9K OHM 1% 1/8W 0805" H 6450 4400 50  0001 C CNN "Description"
 F 5 "Panasonic Electronic Components" H 6450 4400 50  0001 C CNN "Manufacturer"
-F 6 "ERJ-6ENF1004V" H 6450 4400 50  0001 C CNN "Manufacturer Part Number"
+F 6 "ERJ-6ENF4992V" H 6450 4400 50  0001 C CNN "Manufacturer Part Number"
 F 7 "Digi-Key" H 6450 4400 50  0001 C CNN "Supplier"
-F 8 "P1.00MCCT-ND" H 6450 4400 50  0001 C CNN "Supplier Part Number"
+F 8 "P49.9KCCT-ND" H 6450 4400 50  0001 C CNN "Supplier Part Number"
 	1    6450 4400
 	-1   0    0    1
@@
 F 2 "Resistor_SMD:R_0805_2012Metric_Pad1.15x1.40mm_HandSolder" V 6380 3900 50  0001 C CNN
 F 3 "https://industrial.panasonic.com/cdbs/www-data/pdf/RDA0000/AOA0000C304.pdf" H 6450 3900 50  0001 C CNN
-F 4 "" H 6450 3900 50  0001 C CNN "Description"
+F 4 "RES SMD 1.82M OHM 1% 1/8W 0805" H 6450 3900 50  0001 C CNN "Description"
 F 5 "Panasonic Electronic Components" H 6450 3900 50  0001 C CNN "Manufacturer"
-F 6 "ERJ-6ENF1004V" H 6450 3900 50  0001 C CNN "Manufacturer Part Number"
+F 6 "ERJ-6ENF1824V" H 6450 3900 50  0001 C CNN "Manufacturer Part Number"
 F 7 "Digi-Key" H 6450 3900 50  0001 C CNN "Supplier"
-F 8 "P1.00MCCT-ND" H 6450 3900 50  0001 C CNN "Supplier Part Number"
+F 8 "P1.82BTCT-ND" H 6450 3900 50  0001 C CNN "Supplier Part Number"
 	1    6450 3900
 	-1   0    0    1
@@
 F 2 "Resistor_SMD:R_0805_2012Metric_Pad1.15x1.40mm_HandSolder" V 3880 4400 50  0001 C CNN
 F 3 "https://industrial.panasonic.com/cdbs/www-data/pdf/RDA0000/AOA0000C304.pdf" H 3950 4400 50  0001 C CNN
-F 4 "" H 3950 4400 50  0001 C CNN "Description"
+F 4 "RES SMD 49.9K OHM 1% 1/8W 0805" H 3950 4400 50  0001 C CNN "Description"
 F 5 "Panasonic Electronic Components" H 3950 4400 50  0001 C CNN "Manufacturer"
-F 6 "ERJ-6ENF1004V" H 3950 4400 50  0001 C CNN "Manufacturer Part Number"
+F 6 "ERJ-6ENF4992V" H 3950 4400 50  0001 C CNN "Manufacturer Part Number"
 F 7 "Digi-Key" H 3950 4400 50  0001 C CNN "Supplier"
-F 8 "P1.00MCCT-ND" H 3950 4400 50  0001 C CNN "Supplier Part Number"
+F 8 "P49.9KCCT-ND" H 3950 4400 50  0001 C CNN "Supplier Part Number"
 	1    3950 4400
 	-1   0    0    1
@@
 F 2 "Resistor_SMD:R_0805_2012Metric_Pad1.15x1.40mm_HandSolder" V 3880 3900 50  0001 C CNN
 F 3 "https://industrial.panasonic.com/cdbs/www-data/pdf/RDA0000/AOA0000C304.pdf" H 3950 3900 50  0001 C CNN
-F 4 "" H 3950 3900 50  0001 C CNN "Description"
+F 4 "RES SMD 432K OHM 1% 1/8W 0805" H 3950 3900 50  0001 C CNN "Description"
 F 5 "Panasonic Electronic Components" H 3950 3900 50  0001 C CNN "Manufacturer"
-F 6 "ERJ-6ENF1004V" H 3950 3900 50  0001 C CNN "Manufacturer Part Number"
+F 6 "ERJ-6ENF4323V" H 3950 3900 50  0001 C CNN "Manufacturer Part Number"
 F 7 "Digi-Key" H 3950 3900 50  0001 C CNN "Supplier"
-F 8 "P1.00MCCT-ND" H 3950 3900 50  0001 C CNN "Supplier Part Number"
+F 8 "P432KCCT-ND" H 3950 3900 50  0001 C CNN "Supplier Part Number"
 	1    3950 3900
 	-1   0    0    1

Commit message: replace LDO SET resistors with high-precision thin (metal) film variants
Parts:
- R?: Description RES SMD 121K OHM 1% 1/8W 0805 -> RES SMD 121K OHM 0.1% 1/8W 0805 Thin Film; Manufacturer Part Number ERJ-6ENF1213V -> ERA-6AEB1213V; Supplier Part Number P121KCCT-ND -> P121KDACT-ND
Changed lines of the file:
@@
 F 1 "121k" V 4550 4400 50  0000 C CNN
 F 2 "Resistor_SMD:R_0805_2012Metric_Pad1.15x1.40mm_HandSolder" V 4480 4400 50  0001 C CNN
-F 3 "https://industrial.panasonic.com/cdbs/www-data/pdf/RDA0000/AOA0000C304.pdf" H 4550 4400 50  0001 C CNN
-F 4 "RES SMD 121K OHM 1% 1/8W 0805" H 4550 4400 50  0001 C CNN "Description"
+F 3 "https://industrial.panasonic.com/cdbs/www-data/pdf/RDM0000/AOA0000C307.pdf" H 4550 4400 50  0001 C CNN
+F 4 "RES SMD 121K OHM 0.1% 1/8W 0805 Thin Film" H 4550 4400 50  0001 C CNN "Description"
 F 5 "Panasonic Electronic Components" H 4550 4400 50  0001 C CNN "Manufacturer"
-F 6 "ERJ-6ENF1213V" H 4550 4400 50  0001 C CNN "Manufacturer Part Number"
+F 6 "ERA-6AEB1213V" H 4550 4400 50  0001 C CNN "Manufacturer Part Number"
 F 7 "Digi-Key" H 4550 4400 50  0001 C CNN "Supplier"
-F 8 "P121KCCT-ND" H 4550 4400 50  0001 C CNN "Supplier Part Number"
+F 8 "P121KDACT-ND" H 4550 4400 50  0001 C CNN "Supplier Part Number"
 	1    4550 4400
 	1    0    0    1

Commit message: BOM details for LDOs
Parts:
- U?: Description (none) -> 500mA Positive Linear Voltage Regulator; Manufacturer (none) -> Linear Technology; Manufacturer Part Number (none) -> LT3045EMSE#PBF; Supplier (none) -> Digi-Key; Supplier Part Number (none) -> LT3045EMSE#PBF-ND
Changed lines of the file:
@@
 F 2 "Housings_SSOP:MSOP-12-1EP_3x4mm_Pitch0.65mm" H 5500 4400 60  0001 C CNN
 F 3 "https://www.analog.com/media/en/technical-documentation/data-sheets/3045fa.pdf" H 5500 4300 60  0001 C CNN
+F 4 "500mA Positive Linear Voltage Regulator" H 0   0   50  0001 C CNN "Description"
+F 5 "Linear Technology" H 0   0   50  0001 C CNN "Manufacturer"
+F 6 "LT3045EMSE#PBF" H 0   0   50  0001 C CNN "Manufacturer Part Number"
+F 7 "Digi-Key" H 0   0   50  0001 C CNN "Supplier"
+F 8 "LT3045EMSE#PBF-ND" H 0   0   50  0001 C CNN "Supplier Part Number"
 	1    5500 3900
 	1    0    0    -1

Commit message: remove BOM details of copied caps
Parts:
- C? (x2): footprint Capacitor_SMD:C_0805_2012Metric_Pad1.15x1.40mm_HandSolder -> (none); Manufacturer Samsung Electro-Mechanics -> (none); Manufacturer Part Number CL21C4R7BBANNNC -> (none); Supplier Digi-Key -> (none); Supplier Part Number 1276-1832-1-ND -> (none)
Changed lines of the file:
@@
 F 0 "C?" H 4235 4354 50  0000 R CNN
 F 1 "10u" H 4235 4445 50  0000 R CNN
-F 2 "Capacitor_SMD:C_0805_2012Metric_Pad1.15x1.40mm_HandSolder" H 4388 4250 50  0001 C CNN
-F 3 "http://www.samsungsem.com/kr/support/product-search/mlcc/__icsFiles/afieldfile/2018/06/12/CL21C4R7BBANNNC.pdf" H 4350 4400 50  0001 C CNN
+F 2 "" H 4388 4250 50  0001 C CNN
+F 3 "" H 4350 4400 50  0001 C CNN
 F 4 "" H 1900 -750 50  0001 C CNN "Description"
-F 5 "Samsung Electro-Mechanics" H 1900 -750 50  0001 C CNN "Manufacturer"
-F 6 "CL21C4R7BBANNNC" H 1900 -750 50  0001 C CNN "Manufacturer Part Number"
-F 7 "Digi-Key" H 1900 -750 50  0001 C CNN "Supplier"
-F 8 "1276-1832-1-ND" H 1900 -750 50  0001 C CNN "Supplier Part Number"
+F 5 "" H 1900 -750 50  0001 C CNN "Manufacturer"
+F 6 "" H 1900 -750 50  0001 C CNN "Manufacturer Part Number"
+F 7 "" H 1900 -750 50  0001 C CNN "Supplier"
+F 8 "" H 1900 -750 50  0001 C CNN "Supplier Part Number"
 	1    4350 4400
 	1    0    0    1
@@
 F 0 "C?" H 6535 4104 50  0000 R CNN
 F 1 "22u" H 6535 4195 50  0000 R CNN
-F 2 "Capacitor_SMD:C_0805_2012Metric_Pad1.15x1.40mm_HandSolder" H 6688 4000 50  0001 C CNN
-F 3 "http://www.samsungsem.com/kr/support/product-search/mlcc/__icsFiles/afieldfile/2018/06/12/CL21C4R7BBANNNC.pdf" H 6650 4150 50  0001 C CNN
+F 2 "" H 6688 4000 50  0001 C CNN
+F 3 "" H 6650 4150 50  0001 C CNN
 F 4 "" H 4200 -1000 50  0001 C CNN "Description"
-F 5 "Samsung Electro-Mechanics" H 4200 -1000 50  0001 C CNN "Manufacturer"
-F 6 "CL21C4R7BBANNNC" H 4200 -1000 50  0001 C CNN "Manufacturer Part Number"
-F 7 "Digi-Key" H 4200 -1000 50  0001 C CNN "Supplier"
-F 8 "1276-1832-1-ND" H 4200 -1000 50  0001 C CNN "Supplier Part Number"
+F 5 "" H 4200 -1000 50  0001 C CNN "Manufacturer"
+F 6 "" H 4200 -1000 50  0001 C CNN "Manufacturer Part Number"
+F 7 "" H 4200 -1000 50  0001 C CNN "Supplier"
+F 8 "" H 4200 -1000 50  0001 C CNN "Supplier Part Number"
 	1    6650 4150
 	-1   0    0    1
