File: ldo-p12V.sch (KiCad schematic (older format))
At the start: 8 parts

Commit message: fix MSOP12 default lib model path
Parts:
- U?: footprint Housings_SSOP:MSOP-12-1EP_3x4mm_Pitch0.65mm -> Package_SO:MSOP-12-1EP_3x4mm_P0.65mm_EP1.65x2.85mm
Changed lines of the file:
@@
 F 0 "U?" H 6200 4050 60  0000 C CNN
 F 1 "LT3045" H 6200 3950 60  0000 C CNN
-F 2 "Housings_SSOP:MSOP-12-1EP_3x4mm_Pitch0.65mm" H 6200 4450 60  0001 C CNN
+F 2 "Package_SO:MSOP-12-1EP_3x4mm_P0.65mm_EP1.65x2.85mm" H 6200 4450 60  0001 C CNN
 F 3 "https://www.analog.com/media/en/technical-documentation/data-sheets/3045fa.pdf" H 6200 4350 60  0001 C CNN
 F 4 "500mA Positive Linear Voltage Regulator" H 700 50  50  0001 C CNN "Description"
