File: dcdc-bipolar-supply.sch (KiCad schematic (older format))
At the start: 14 parts

Commit message: add footprint for schottky diodes
Parts:
- D? (x4): footprint (none) -> Diode_SMD:D_SOD-123
Changed lines of the file:
@@
 F 0 "D?" V 5454 3379 50  0000 L CNN
 F 1 "20V/500mA" V 5545 3379 50  0000 L CNN
-F 2 "" H 5500 3300 50  0001 C CNN
+F 2 "Diode_SMD:D_SOD-123" H 5500 3300 50  0001 C CNN
 F 3 "https://www.onsemi.cn/PowerSolutions/document/MBR0520L-D.pdf" H 5500 3300 50  0001 C CNN
 F 4 "SCHOTTKY 20V 500MA SOD123" H 0   0   50  0001 C CNN "Description"
@@
 F 0 "D?" H 5750 2834 50  0000 C CNN
 F 1 "20V/500mA" H 5750 2925 50  0000 C CNN
-F 2 "" H 5750 3050 50  0001 C CNN
+F 2 "Diode_SMD:D_SOD-123" H 5750 3050 50  0001 C CNN
 F 3 "https://www.onsemi.cn/PowerSolutions/document/MBR0520L-D.pdf" H 5750 3050 50  0001 C CNN
 F 4 "SCHOTTKY 20V 500MA SOD123" H 0   0   50  0001 C CNN "Description"
@@
 F 0 "D?" V 5454 4721 50  0000 R CNN
 F 1 "20V/500mA" V 5545 4721 50  0000 R CNN
-F 2 "" H 5500 4800 50  0001 C CNN
+F 2 "Diode_SMD:D_SOD-123" H 5500 4800 50  0001 C CNN
 F 3 "https://www.onsemi.cn/PowerSolutions/document/MBR0520L-D.pdf" H 5500 4800 50  0001 C CNN
 F 4 "SCHOTTKY 20V 500MA SOD123" H 0   0   50  0001 C CNN "Description"
@@
 F 0 "D?" H 5750 5250 50  0000 C CNN
 F 1 "20V/500mA" H 5750 5150 50  0000 C CNN
-F 2 "" H 5750 5050 50  0001 C CNN
+F 2 "Diode_SMD:D_SOD-123" H 5750 5050 50  0001 C CNN
 F 3 "https://www.onsemi.cn/PowerSolutions/document/MBR0520L-D.pdf" H 5750 5050 50  0001 C CNN
 F 4 "SCHOTTKY 20V 500MA SOD123" H 0   0   50  0001 C CNN "Description"
